File: pcb/my-keeb/my-keeb.kicad_sch (KiCad schematic)
At the start: 63 parts, among them SW1 SW_Push, SW10 SW_Push, SW11 SW_Push, SW12 SW_Push, SW13 SW_Push, SW14 SW_Push, SW15 SW_Push, SW16 SW_Push, SW19 SW_Push, SW2 SW_Push, SW20 SW_Push, SW21 SW_Push, SW22 SW_Push, SW23 SW_Push, SW24 SW_Push, SW25 SW_Push, SW26 SW_Push, SW27 SW_Push, SW28 SW_Push, SW29 SW_Push, SW3 SW_Push, SW30 SW_Push, SW31 SW_Push, SW32 SW_Push, SW4 SW_Push, SW5 SW_Push, SW6 SW_Push, SW7 SW_Push, SW8 SW_Push, SW9 SW_Push

Commit message: Starting laying footprints on pcb
Parts:
- removed A1: RaspberryPi_Pico, Module:RaspberryPi_Pico_Common_Unspecified, symbol MCU_Module:RaspberryPi_Pico
- removed D1, D3: 1N4148, Diode_THT:D_DO-35_SOD27_P7.62mm_Horizontal, symbol Diode:1N4148
- removed S1: MX_stab, PCM_marbastlib-mx:STAB_MX_P_6.25u, symbol PCM_marbastlib-mx:MX_stab
- removed SW1, SW3: SW_Push, symbol Switch:SW_Push
- added H1, H2, H3, H4, H5, H6: MountingHole, symbol Mechanical:MountingHole
- added S2, S3, S4, S5: MX_stab, PCM_marbastlib-mx:STAB_MX_3u, symbol PCM_marbastlib-mx:MX_stab
- A2: footprint Module:RaspberryPi_Pico_Common_Unspecified -> Module:RaspberryPi_Pico_Common_THT
- SW10, SW11, SW12, SW13, SW14, SW15, SW16, SW19, SW2, SW20, SW21, SW22, SW23, SW24, SW25, SW26, SW27, SW28, SW29, SW30, SW31, SW32, SW4, SW5, SW6, SW7, SW8, SW9: footprint (none) -> PCM_marbastlib-mx:SW_MX_1u
