File: pcb/my-keeb/my-keeb.kicad_pcb (KiCad board)
At the start: 2 copper layers, 235.4 x 97.4 mm, 152 parts, among them SW10 SW_Push, SW11 SW_Push, SW12 SW_Push, SW13 SW_Push, SW14 SW_Push, SW15 SW_Push, SW16 SW_Push, SW17 SW_Push, SW18 SW_Push, SW19 SW_Push, SW2 SW_Push, SW20 SW_Push, SW21 SW_Push, SW22 SW_Push, SW23 SW_Push, SW24 SW_Push, SW25 SW_Push, SW26 SW_Push, SW27 SW_Push, SW28 SW_Push, SW29 SW_Push, SW3 SW_Push, SW30 SW_Push, SW31 SW_Push, SW32 SW_Push, SW33 SW_Push, SW34 SW_Push, SW35 SW_Push, SW36 SW_Push, SW37 SW_Push, SW38 SW_Push, SW39 SW_Push, SW4 SW_Push, SW40 SW_Push, SW41 SW_Push, SW42 SW_Push, SW43 SW_Push, SW44 SW_Push, SW45 SW_Push, SW46 SW_Push, SW47 SW_Push, SW48 SW_Push, SW49 SW_Push, SW5 SW_Push, SW50 SW_Push, SW51 SW_Push, SW52 SW_Push, SW53 SW_Push, SW54 SW_Push, SW55 SW_Push, SW56 SW_Push, SW58 SW_Push, SW59 SW_Push, SW6 SW_Push, SW60 SW_Push, SW61 SW_Push, SW63 SW_Push, SW64 SW_Push, SW65 SW_Push, SW66 SW_Push, SW68 SW_Push, SW69 SW_Push, SW7 SW_Push, SW70 SW_Push, SW72 SW_Push, SW8 SW_Push, SW9 SW_Push

Commit message: Placing the components
Parts:
- removed D17, D18, D3, D33, D34, D35, D36, D37, D38, D39, D40, D41, D42, D43, D44, D45, D46, D47, D48, D49, D50, D51, D52, D53, D54, D55, D56, D58, D59, D60, D61, D63, D64, D65, D66, D68, D69, D70, D72 (x2): 1N4148, Diode_THT:D_DO-35_SOD27_P7.62mm_Horizontal
- removed the D2 at (69.3, -164.4)
- removed the D2 at (62.5, 85.3)
- removed the D2 at (62.5, 28.1)
- removed the D2 at (172.9, 28.3)
- removed the D2 at (531.5, 39.6)
- removed the S2 at (53.0, 24.0)
- removed the S2 at (522.0, 35.5)
- removed the S2 at (53.0, 81.2)
- removed the S4 at (239.5, -68.5)
- removed the S4 at (303.2, -125.9)
- removed SW17, SW18, SW3, SW33, SW34, SW35, SW36, SW37, SW38, SW39, SW40, SW41, SW42, SW43, SW44, SW45, SW46, SW47, SW48, SW49, SW50, SW51, SW52, SW53, SW54, SW55, SW56, SW58, SW59, SW60, SW61, SW63, SW64, SW65, SW66, SW68, SW69, SW70, SW72 (x2): SW_Push, PCM_marbastlib-mx:SW_MX_1u
- removed the SW2 at (163.4, 24.2)
- removed the SW2 at (522.0, 35.5)
- removed the SW2 at (59.8, -168.5)
- removed the SW2 at (53.0, 24.0)
- removed the SW2 at (53.0, 81.3)
- added D2: 1N4148, Diode_THT:D_DO-35_SOD27_P7.62mm_Horizontal, F.Cu at (-211.9, -124.8)
- added S2: MX_stab, PCM_marbastlib-mx:STAB_MX_3u, F.Cu at (-183.4, -128.6)
- added S4: MX_stab, PCM_marbastlib-mx:STAB_MX_3u, F.Cu at (-88.1, -71.4)
- added SW2: SW_Push, Button_Switch_Keyboard:SW_Cherry_MX_1.00u_PCB, F.Cu at (-218.9, -133.7)
- SW10, SW11, SW12, SW13, SW14, SW15, SW16, SW19, SW20, SW21, SW22, SW23, SW24, SW25, SW26, SW27, SW28, SW29, SW30, SW31, SW32, SW4, SW5, SW6, SW7, SW8, SW9: footprint PCM_marbastlib-mx:SW_MX_1u -> Button_Switch_Keyboard:SW_Cherry_MX_1.00u_PCB
- moved D13 719.7 mm to (-173.8, -67.6), turned to 90 degrees
- moved D4 710.0 mm to (-211.9, -105.7), turned to 90 degrees
- moved D5 705.3 mm to (-211.9, -86.7), turned to 90 degrees
- moved D6 700.9 mm to (-211.9, -67.6), turned to 90 degrees
- moved D7 695.4 mm to (-192.9, -105.7), turned to 90 degrees
- moved D8 690.4 mm to (-192.9, -86.7), turned to 90 degrees
- moved D10 688.3 mm to (-173.8, -124.8), turned to 90 degrees
- moved D9 685.6 mm to (-192.9, -67.6), turned to 90 degrees
- moved D11 682.6 mm to (-173.8, -105.7), turned to 90 degrees
- moved D12 677.1 mm to (-173.8, -86.7), turned to 90 degrees
- moved D14 666.1 mm to (-154.8, -105.7), turned to 90 degrees
- moved D15 661.1 mm to (-154.8, -86.7), turned to 90 degrees
- moved SW4 648.9 mm to (-218.9, -114.6)
- moved SW5 647.9 mm to (-218.9, -95.6)
- moved SW6 646.9 mm to (-218.9, -76.5)
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Other:
- board size 235.4 x 97.4 mm -> 233.4 x 85.7 mm

Commit message: Added routing traces
Parts:
- moved D14 19.1 mm to (-173.8, -105.7)
- moved D15 19.1 mm to (-173.8, -86.7)
- moved D7 19.1 mm to (-211.9, -105.7)
- moved D8 19.1 mm to (-211.9, -86.7)
- moved D9 19.1 mm to (-211.9, -67.6)
- moved D26 19.1 mm to (-40.5, -105.7)
- moved D27 19.1 mm to (-40.5, -86.7)
- moved D28 19.1 mm to (-40.5, -67.6)
- moved D20 19.0 mm to (-78.6, -105.7)
- moved D21 19.0 mm to (-78.6, -86.7)
- moved D22 19.0 mm to (-59.5, -124.8)
- moved D23 19.0 mm to (-59.5, -105.7)
- moved D24 19.0 mm to (-59.5, -86.7)
- moved D25 19.0 mm to (-59.5, -67.6)
- moved D29 19.0 mm to (-21.4, -124.8)
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Routing:
- net /ROW3: track 0.00 -> 333.2 mm
- net /ROW2: track 0.00 -> 327.0 mm
- net /ROW1: track 0.00 -> 259.6 mm
- net /ROW0: track 0.00 -> 244.5 mm
- net /COL8: track 0.00 -> 209.5 mm
- net /COL9: track 0.00 -> 197.5 mm
- net /COL7: track 0.00 -> 182.0 mm
- net /COL0: track 0.00 -> 164.5 mm
- net /COL1: track 0.00 -> 150.2 mm
- net /COL6: track 0.00 -> 140.9 mm
- net /COL2: track 0.00 -> 130.4 mm
- net /COL5: track 0.00 -> 101.7 mm
- net /<NO NET>: track 0.00 -> 56.8 mm
- net /COL4: track 0.00 -> 54.3 mm
- net Net-(D2-A): track 0.00 -> 6.53 mm
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- added copper zone on B.Cu, net (none)
- added copper zone on F.Cu, net (none)
Other:
- board size 233.4 x 85.7 mm -> 234.5 x 85.7 mm

Commit message: Added mountingholes and made gerbers
Parts:
- added REF**: MountingHole_2.2mm_M2, MountingHole:MountingHole_2.2mm_M2, F.Cu at (0.00, -142.0)
- added REF**: MountingHole_2.2mm_M2, MountingHole:MountingHole_2.2mm_M2, F.Cu at (0.00, -57.1)
- added REF**: MountingHole_2.2mm_M2, MountingHole:MountingHole_2.2mm_M2, F.Cu at (-116.7, -57.1)
- added REF**: MountingHole_2.2mm_M2, MountingHole:MountingHole_2.2mm_M2, F.Cu at (-233.4, -142.0)
- added REF**: MountingHole_2.2mm_M2, MountingHole:MountingHole_2.2mm_M2, F.Cu at (-233.4, -58.0)
Routing:
- net /ROW3: track 333.2 -> 409.4 mm
- net /ROW1: track 259.6 -> 317.7 mm
- net /COL9: track 197.5 -> 254.6 mm
- net /COL7: track 182.0 -> 234.6 mm
- net /COL8: track 209.5 -> 247.6 mm
- net /ROW0: track 244.5 -> 281.7 mm
- net /COL6: track 140.9 -> 160.0 mm
- net /COL2: track 130.4 -> 127.5 mm
- net /ROW2: track 327.0 -> 327.9 mm
- removed copper zone on B.Cu, net (none)
- removed copper zone on F.Cu, net (none)
Other:
- board size 234.5 x 85.7 mm -> 242.8 x 92 mm
